File: hand-sanitizer.kicad_pcb (KiCad board)
At the start: 2 copper layers, 61.3 x 46.7 mm, 29 parts, among them J1 Conn_01x02, J2 prog, J3 Conn_01x06, J4 relay_terminal_out, K1 Milon-Relay, Q1 MMBT2222, SW1 SW_Push, U1 ATmega8A-AU, U2 L78L05_SOT89

Commit message: Minor changes to pcb
Other:
- board text added: "<- connect these two points via a bridge ->"
